File: hardware/imu.kicad_sch (KiCad schematic)
At the start: 4 parts, among them U9 LSM6DSV16XTR

Commit message: Swap 1.8V LDO and IMU, fix BOM/CPL export hygiene
Mirrors the same pass done on OpenFC-Lite-Mini.

Part changes:
- NCV8187AMT180TAG (stock 0 at JLC) replaced by U15 LP5912-1.8DRVR
  (C2876234), same WSON-6 2x2 land pattern as the LP5912-3.3, PG retained.
- U9 LSM6DSV16XTR replaced by BMI270 (C2836813) in the schematic. Bosch
  Table 22 matches the existing LGA-14 symbol pin for pin, so no rewire.

Export fixes:
- U15, CN1 and U13 carried their part numbers in a field named "LCSC Part"
  rather than "LCSC" and exported blank. Renamed. CN1 (C160404) and U13
  (C160403) are real JST connectors and stay in the BOM.
- J3, J6, J10, J16, J19, J23 (lib:small_pad) and TP1 to TP4 (TestPoint) were
  still reaching the BOM with no part number. Set to in_bom=no, on_board=yes,
  dnp=no: copper stays, BOM entry goes.
- 57 pad and testpoint footprints now carry exclude_from_bom plus
  exclude_from_pos_files instead of the dnp flag. Previously 47 pads leaked
  into the position file on every export.

BOM and CPL now agree at 111 placements with no blank part numbers, exported
without any dnp flag. ERC is unchanged against HEAD (198 vs 199 violations,
all pre-existing).

Known outstanding, not in this commit: C32 is still C105226 while C42 is
C415703, and the PCB copy of U9 still carries the LSM6 part number until
Update PCB from Schematic is run. The panel file is deleted in the working
tree pending a rebuild and is deliberately left uncommitted.

Co-Authored-By: Claude Fable 5 <noreply@anthropic.com>
Parts:
- U9: value LSM6DSV16XTR -> BMI270; LCSC C5267406 -> C2836813; MPN LSM6DSV16XTR -> BMI270; Manufacturer STMicroelectronics -> Bosch
Changed lines of the file:
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@@
 			)
 		)
-		(property "Value" "LSM6DSV16XTR"
+		(property "Value" "BMI270"
 			(at 60.96 70.866 0)
 			(show_name no)
@@
 			)
 		)
-		(property "LCSC" "C5267406"
+		(property "LCSC" "C2836813"
 			(at 72.39 87.63 0)
 			(hide yes)
@@
 			)
 		)
-		(property "MPN" "LSM6DSV16XTR"
+		(property "MPN" "BMI270"
 			(at 0 0 0)
 			(hide yes)
@@
 			)
 		)
-		(property "Manufacturer" "STMicroelectronics"
+		(property "Manufacturer" "Bosch"
 			(at 0 0 0)
 			(hide yes)
