File: hardware/pads.kicad_sch (KiCad schematic)
At the start: 60 parts, among them CN1 SM04B-SRSS-TB, J1 5V, J10 5V, J11 5V, J12 5V, J13 5V, J14 5V, J15 5V, J16 5V, J17 5V, J18 5V, J19 5V, J2 5V, J20 5V, J21 5V, J22 5V, J23 5V, J24 5V, J25 5V, J26 5V, J27 5V, J28 5V, J29 5V, J3 5V, J30 5V, J31 5V, J32 5V, J33 5V, J34 5V, J35 5V, J36 5V, J37 5V, J38 5V, J39 5V, J4 5V, J40 5V, J41 5V, J42 5V, J43 5V, J44 5V, J45 5V, J46 5V, J47 5V, J48 5V, J49 5V, J5 5V, J50 5V, J51 5V, J52 5V, J53 5V, J54 5V, J55 5V, J6 5V, J7 5V, J8 5V, J9 5V, P1 SM08B-SRSS-TB(LF)(SN), U13 SM03B-SRSS-TB, U14 SM06B-SRSS-TB(LF)(SN), U8 SM06B-SRSS-TB(LF)(SN)

Commit message: Swap 1.8V LDO and IMU, fix BOM/CPL export hygiene
Mirrors the same pass done on OpenFC-Lite-Mini.

Part changes:
- NCV8187AMT180TAG (stock 0 at JLC) replaced by U15 LP5912-1.8DRVR
  (C2876234), same WSON-6 2x2 land pattern as the LP5912-3.3, PG retained.
- U9 LSM6DSV16XTR replaced by BMI270 (C2836813) in the schematic. Bosch
  Table 22 matches the existing LGA-14 symbol pin for pin, so no rewire.

Export fixes:
- U15, CN1 and U13 carried their part numbers in a field named "LCSC Part"
  rather than "LCSC" and exported blank. Renamed. CN1 (C160404) and U13
  (C160403) are real JST connectors and stay in the BOM.
- J3, J6, J10, J16, J19, J23 (lib:small_pad) and TP1 to TP4 (TestPoint) were
  still reaching the BOM with no part number. Set to in_bom=no, on_board=yes,
  dnp=no: copper stays, BOM entry goes.
- 57 pad and testpoint footprints now carry exclude_from_bom plus
  exclude_from_pos_files instead of the dnp flag. Previously 47 pads leaked
  into the position file on every export.

BOM and CPL now agree at 111 placements with no blank part numbers, exported
without any dnp flag. ERC is unchanged against HEAD (198 vs 199 violations,
all pre-existing).

Known outstanding, not in this commit: C32 is still C105226 while C42 is
C415703, and the PCB copy of U9 still carries the LSM6 part number until
Update PCB from Schematic is run. The panel file is deleted in the working
tree pending a rebuild and is deliberately left uncommitted.

Co-Authored-By: Claude Fable 5 <noreply@anthropic.com>
Parts:
- CN1: LCSC (none) -> C160404; LCSC Part C160404 -> (none)
- J10, J16, J19, J23, J3, J6: now left out of the parts list
- U13: LCSC (none) -> C160403; LCSC Part C160403 -> (none)

Commit message: 4V5 rework: TPS2116 mux replaced by DSK24 diode-OR
U5, its RB161QS diodes, R19/R20 and C28 removed. D6 from the buck
output and D10 from +5V_USB feed the new +4v5 net, which supplies the
3.3 V and 1.8 V LDOs, the 6-pin JST and the J5/J47 pads. The buck
output is plain +5V and drives the external 5 V pads directly. All 596
vias at 0.35/0.2, so the line-standard floors pass. DSK24 footprint and
3D model committed with the change. DRC severity choices per Stan.

Co-Authored-By: Claude Opus 5 (1M context) <noreply@anthropic.com>
Connections:
- net +5V: no longer J47.1 (Pin_1), J5.1 (Pin_1), U14.1
- new net +4v5: J47.1 (Pin_1), J5.1 (Pin_1), U14.1
