File: hardware/rp2350a.kicad_sch (KiCad schematic)
At the start: 48 parts, among them Q1 AP1606, Q2 AP1606, U1 TS2306A 240GF MSM 9_C2976675, U2 RP2354B_C39843328, X1 XTM25012000JT00351001

Commit message: 4V5 rework: TPS2116 mux replaced by DSK24 diode-OR
U5, its RB161QS diodes, R19/R20 and C28 removed. D6 from the buck
output and D10 from +5V_USB feed the new +4v5 net, which supplies the
3.3 V and 1.8 V LDOs, the 6-pin JST and the J5/J47 pads. The buck
output is plain +5V and drives the external 5 V pads directly. All 596
vias at 0.35/0.2, so the line-standard floors pass. DSK24 footprint and
3D model committed with the change. DRC severity choices per Stan.

Co-Authored-By: Claude Opus 5 (1M context) <noreply@anthropic.com>
Connections:
- net +5V renamed +4v5
Changed lines of the file:
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@@
+	)
+	(symbol
+		(lib_id "power:+5V")
+		(at 425.45 275.59 0)
+		(unit 1)
+		(body_style 1)
+		(exclude_from_sim no)
+		(in_bom yes)
+		(on_board yes)
+		(in_pos_files yes)
+		(dnp no)
+		(fields_autoplaced yes)
+		(property "Reference" "#PWR081"
+			(at 425.45 279.4 0)
+			(hide yes)
+			(show_name no)
+			(do_not_autoplace no)
+			(effects
+				(font
+					(size 1.27 1.27)
+				)
+			)
+		)
+		(property "Value" "+4v5"
+			(at 425.45 270.51 0)
+			(show_name no)
+			(do_not_autoplace no)
+			(effects
+				(font
+					(size 1.27 1.27)
+				)
+			)
+		)
+		(property "Footprint" ""
+			(at 425.45 275.59 0)
+			(hide yes)
+			(show_name no)
+			(do_not_autoplace no)
+			(effects
+				(font
+					(size 1.27 1.27)
+				)
+			)
+		)
+		(property "Datasheet" ""
+			(at 425.45 275.59 0)
+			(hide yes)
+			(show_name no)
+			(do_not_autoplace no)
+			(effects
+				(font
+					(size 1.27 1.27)
+				)
+			)
+		)
+		(property "Description" "Power symbol creates a global label with name \"+5V\""
+			(at 425.45 275.59 0)
+			(hide yes)
+			(show_name no)
+			(do_not_autoplace no)
+			(effects
+				(font
+					(size 1.27 1.27)
+				)
+			)
+		)
+		(pin "1"
+		)
+		(instances
+			(project "OpenFC"
+				(path "/fb88b6f9-ee39-4640-a9d4-04a17ceeac64/cec45a0d-1d48-4800-9760-14c521e5fc8b"
+					(reference "#PWR081")
+					(unit 1)
+				)
+			)
+		)
 	)
 	(symbol
@@
 					(unit 1)
 				)
-			)
-		)
-	)
-	(symbol
-		(lib_id "power:+5V")
-		(at 425.45 275.59 0)
-		(unit 1)
-		(body_style 1)
-		(exclude_from_sim no)
-		(in_bom yes)
-		(on_board yes)
-		(in_pos_files yes)
-		(dnp no)
-		(fields_autoplaced yes)
-		(property "Reference" "#PWR057"
-			(at 425.45 279.4 0)
-			(hide yes)
-			(show_name no)
-			(do_not_autoplace no)
-			(effects
-				(font
-					(size 1.27 1.27)
-				)
-			)
-		)
-		(property "Value" "+5V"
-			(at 425.45 270.51 0)
-			(show_name no)
-			(do_not_autoplace no)
-			(effects
-				(font
-					(size 1.27 1.27)
-				)
-			)
-		)
-		(property "Footprint" ""
-			(at 425.45 275.59 0)
-			(hide yes)
-			(show_name no)
-			(do_not_autoplace no)
-			(effects
-				(font
-					(size 1.27 1.27)
-				)
-			)
-		)
-		(property "Datasheet" ""
-			(at 425.45 275.59 0)
-			(hide yes)
-			(show_name no)
-			(do_not_autoplace no)
-			(effects
-				(font
-					(size 1.27 1.27)
-				)
-			)
-		)
-		(property "Description" "Power symbol creates a global label with name \"+5V\""
-			(at 425.45 275.59 0)
-			(hide yes)
-			(show_name no)
-			(do_not_autoplace no)
-			(effects
-				(font
-					(size 1.27 1.27)
-				)
-			)
-		)
-		(pin "1"
-		)
-		(instances
-			(project "OpenFC"
-				(path "/fb88b6f9-ee39-4640-a9d4-04a17ceeac64/cec45a0d-1d48-4800-9760-14c521e5fc8b"
-					(reference "#PWR057")
-					(unit 1)
-				)

Commit message: schematics: complete Manufacturer/MPN coverage, trim stray whitespace
16 field fixes: Manufacturer backfilled from the LCSC catalogue on osd,
power and rp2350a sheets, trailing space trimmed from four XL-1005UGC MPNs.
Part of the fab-agnostic BOM standardisation for quoting outside JLCPCB.

kicad-skip reflowed the touched files; structural diff against the originals
shows only property changes, ERC identical (179 violations before and after).

Co-Authored-By: Claude Fable 5 <noreply@anthropic.com>
Parts:
- R18: MPN (none) -> RTT012401FTH; Manufacturer (none) -> RALEC
