File: hardware/OpenFC.kicad_pcb (KiCad board)
At the start: 6 copper layers, 37.9 x 37.9 mm, 164 parts, among them CN1 SM04B-SRSS-TB, J1 5V, J10 5V, J11 5V, J12 5V, J13 5V, J14 5V, J15 5V, J16 5V, J17 5V, J18 5V, J19 5V, J2 5V, J20 5V, J21 5V, J22 5V, J23 5V, J24 5V, J25 5V, J26 5V, J27 5V, J28 5V, J29 5V, J3 5V, J30 5V, J31 5V, J32 5V, J33 5V, J34 5V, J35 5V, J36 5V, J37 5V, J38 5V, J39 5V, J4 5V, J40 5V, J41 5V, J42 5V, J43 5V, J44 5V, J47 5V, J48 5V, J49 5V, J5 5V, J50 5V, J51 5V, J52 5V, J53 5V, J54 5V, J55 5V, J6 5V, J7 5V, J8 5V, J9 5V, P1 SM08B-SRSS-TB(LF)(SN), Q1 AP1606, Q2 AP1606, U1 TS2306A 240GF MSM 9_C2976675, U10 SN74LVC1G3157DTBR, U11 COS8051SOT, U12 TLV7031DPWR, U13 SM03B-SRSS-TB, U14 SM06B-SRSS-TB(LF)(SN), U15 LP5912-1.8DRVR, U16 LMR51635YDDCR, U2 RP2354B_C39843328, U6 LMR51635YDDCR, U7 LP5912-3.3DRVR, U8 SM06B-SRSS-TB(LF)(SN), U9 BMI270, X1 XTM25012000JT00351001

Commit message: AGENTS: record rev3.3; rev silk synced by pipeline
Co-Authored-By: Claude Fable 5 <noreply@anthropic.com>
Other:
- board text added: "REV3.3"
- board text removed: "REV3.1"
Changed lines of the file:
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@@
 	)
 	(paper "A4")
+	(title_block
+		(rev "rev3.3")
+	)
 	(layers
 		(0 "F.Cu" signal)
@@
 		)
 	)
-	(gr_text "REV3.1"
+	(gr_text "REV3.3"
 		(at 166.11 76.31 0)
 		(layer "B.SilkS")
@@
 			(justify left bottom mirror)
 		)
-		(render_cache "REV3.1" 0
+		(render_cache "REV3.3" 0
 			(polygon
 				(pts
@@
 			(polygon
 				(pts
-					(xy 163.682531 76.14) (xy 163.850265 76.14) (xy 163.850265 75.237644) (xy 163.767894 75.155212)
-					(xy 163.682531 75.155212)
+					(xy 163.715687 76.14) (xy 163.753836 76.135324) (xy 163.787139 76.121687) (xy 163.816803 76.098722)
+					(xy 163.839765 76.069057) (xy 163.853403 76.035735) (xy 163.85808 75.997545) (xy 163.85808 75.808806)
+					(xy 163.690347 75.808806) (xy 163.690347 75.972144) (xy 163.611884 75.972144) (xy 163.611884 75.793907)
+					(xy 163.61648 75.769738) (xy 163.630385 75.748845) (xy 163.651013 75.734495) (xy 163.676181 75.729672)
+					(xy 163.77687 75.729672) (xy 163.77687 75.561816) (xy 163.676181 75.561816) (xy 163.650942 75.557068)
+					(xy 163.630385 75.543009) (xy 163.616473 75.52242) (xy 163.611884 75.498618) (xy 163.611884 75.323068)
+					(xy 163.690347 75.323068) (xy 163.690347 75.483902) (xy 163.85808 75.483902) (xy 163.85808 75.296568)
+					(xy 163.853409 75.258714) (xy 163.839778 75.225675) (xy 163.816803 75.196245) (xy 163.787157 75.173427)
+					(xy 163.753853 75.159864) (xy 163.715687 75.155212) (xy 163.586543 75.155212) (xy 163.54929 75.159819)
+					(xy 163.516197 75.173354) (xy 163.48616 75.196306) (xy 163.462748 75.225827) (xy 163.448892 75.258904)
+					(xy 163.44415 75.296751) (xy 163.44415 75.506189) (xy 163.448951 75.544036) (xy 163.462995 75.577129)
+					(xy 163.48677 75.606695) (xy 163.525971 75.645774) (xy 163.48677 75.685158) (xy 163.463011 75.714922)
+					(xy 163.448958 75.748278) (xy 163.44415 75.786458) (xy 163.44415 75.997362) (xy 163.448897 76.035545)
+					(xy 163.462761 76.068905) (xy 163.48616 76.098661) (xy 163.516214 76.12176) (xy 163.549306 76.13537)
+					(xy 163.586543 76.14)
 				)
 			)
